File: DP3EXB.kicad_pcb (KiCad board)
At the start: 4 copper layers, 41.3 x 18.3 mm, 58 parts, among them J1 Conn_01x16_Pin, J2 Conn_01x16_Pin, J3 Conn_01x06_Pin, U1 ATSAME51G19A-MF, U2 MCP2542FDT-E/MNY, U3 AP2112K-3.3TRG1, U4 SN74AHCT541PWR, X1 TSX-3225 25.0000MF10P-C

Commit message: Minor updates
Minor updates
Routing:
- net V33: track 26.2 -> 27.2 mm
- net GND: track 53.2 -> 53.9 mm
- net PB09: track 18.6 -> 18.0 mm
- net PB08: track 17.3 -> 16.7 mm
