File: DP3EXB.kicad_pcb (KiCad board)
At the start: 4 copper layers, 41.3 x 18.3 mm, 58 parts, among them J1 Conn_01x16_Pin, J2 Conn_01x16_Pin, J3 Conn_01x06_Pin, U1 ATSAME51G19A-MF, U2 MCP2542FDT-E/MNY, U3 AP2112K-3.3TRG1, U4 SN74AHCT541PWR, X1 TSX-3225 25.0000MF10P-C

Commit message: Minor updates
Minor updates
Routing:
- net PA08: track 13.7 -> 13.1 mm
Other:
- board text added: "3.3V"
- board text added: "CAN"
- board text added: "CAN_H"
- board text added: "CAN_L"
- board text added: "DP3EXB V0.1"
- board text added: "PA00"
- board text added: "PA01"
- board text added: "PA04"
- board text added: "PA05"
- board text added: "PA06"
- board text added: "PA07"
- board text added: "PA08"
- board text added: "PA09"
- board text added: "PA10"
- board text added: "PA11"
- board text added: "PA12"
- board text added: "PA13"
- board text added: "PA16"
- board text added: "PA17"
- board text added: "PA18"
- board text added: "PA19"
- board text added: "PA20"
- board text added: "PA21"
- board text added: "PA24"
- board text added: "PA25"
- board text added: "PA27"
- board text added: "PB02"
- board text added: "PB08"
- board text added: "PB09"
- board text added: "PB10"
- board text added: "PB11"
- board text added: "PB23"
- board text added: "https://github.com/jcwebber93/DP3EXB"
- board text removed: "https://github.com/jcwebber93/DP3EXB DP3EXB V0.1"
